File: micromouse-hardware.kicad_sch (KiCad schematic)
At the start: 58 parts, among them J1 BATT-CONN, Q1 BCP56, Q10 BCP56, Q2 BCP56, Q3 BCP56, Q4 TEFT4300, Q5 TEFT4300, Q6 TEFT4300, Q7 TEFT4300, Q8 TEFT4300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

Commit message: promjenio tranistore u mosfete, jos neki popravci
Parts:
- removed Q1, Q10, Q2, Q3, Q9: BCP56, Custom:SOT-223-3_TabPin4, symbol Transistor_BJT:BCP56
- removed R10, R13, R2, R4, R7: 820R, Resistor_SMD:R_0603_1608Metric, symbol Device:R
- removed R11, R14, R3, R5, R8: 10K, Resistor_SMD:R_0603_1608Metric, symbol Device:R
- removed U5: LM2575GR-5.0, Package_TO_SOT_SMD:TO-263-5_TabPin3, symbol Regulator_Switching:LM2575-5.0BU
- added C8, C9: 100nF, Capacitor_SMD:C_0805_2012Metric_Pad1.18x1.45mm_HandSolder, symbol Device:C
- added IC1: LM2575SX-5.0_NOPB, Custom:KTT0005B, symbol LM2575SX-5_0_NOPB:LM2575SX-5.0_NOPB
- added IC2: TBD62003AFG,EL, SOIC127P630X190-16N, symbol TBD62003AFG_EL:TBD62003AFG,EL
- A1, ME1, ME2: now left out of the parts list
- C1: footprint Capacitor_SMD:C_0603_1608Metric -> Capacitor_SMD:C_0805_2012Metric_Pad1.18x1.45mm_HandSolder; Manufacturer_Part_Number (none) -> MCASL21GBB7106KTNA01
- C2: footprint Capacitor_SMD:C_0603_1608Metric -> Capacitor_SMD:C_0805_2012Metric_Pad1.18x1.45mm_HandSolder; Manufacturer_Part_Number (none) -> KAF21KR71E225KU
- C3: footprint Capacitor_SMD:C_0603_1608Metric -> Capacitor_SMD:C_0805_2012Metric_Pad1.18x1.45mm_HandSolder; Manufacturer_Part_Number (none) -> KAF21BR72A103JT
- C4, C6: Manufacturer_Part_Number (none) -> EDK477M016A9MAA
- C5, C7: footprint Capacitor_SMD:C_0603_1608Metric -> Capacitor_SMD:C_0805_2012Metric_Pad1.18x1.45mm_HandSolder; Manufacturer_Part_Number (none) -> KAM21BR71H104JM
- D1, D2, D3, D4, D5: value SHF4545 -> SFH4545; Manufacturer_Part_Number (none) -> SFH 4545
- D8: Manufacturer_Part_Number (none) -> SS26SHE3_B/H
- L1: Manufacturer_Part_Number (none) -> SRR1280-221K
- Q4, Q5, Q6, Q7, Q8: Manufacturer_Part_Number (none) -> TEFT4300
- R1, R12, R15, R6, R9: footprint Resistor_SMD:R_0603_1608Metric -> Resistor_SMD:R_0805_2012Metric_Pad1.20x1.40mm_HandSolder; Manufacturer_Part_Number (none) -> CRGS0805J33R
- R16, R17, R18, R19, R20: Manufacturer_Part_Number (none) -> SFR25H0001801JA500
- R23, R24: footprint Resistor_SMD:R_0603_1608Metric -> Resistor_SMD:R_0805_2012Metric_Pad1.20x1.40mm_HandSolder; Manufacturer_Part_Number (none) -> CHP0805-FX-1002ELF
- SW2: Manufacturer_Part_Number (none) -> 206-2ST
- SW3: Manufacturer_Part_Number (none) -> EG1218
- U1: Manufacturer_Part_Number (none) -> DRV8833CPWPR
- U2: footprint Package_SO:SOIC-16_4.55x10.3mm_P1.27mm -> Package_SO:SOIC-16_3.9x9.9mm_P1.27mm; Manufacturer_Part_Number (none) -> CD74HC4051M
- U3: Manufacturer_Part_Number (none) -> 74HC238D
Connections:
- net +5V: now also C8.1, C9.1, IC1.4 (FEEDBACK), IC2.9 (COMMON)
- net +VBAT: now also IC1.1 (VIN)
- net GND: now also C8.2, C9.2, IC1.3 (GND), IC1.5 (~{ON_}/_OFF), IC1.6 (TAB_(GND)), IC2.8 (GND)
- net at R15.2: now also IC2.12 (O5)
- net at U3.11 (Y4): now also IC2.5 (I5)
- net at U3.14 (Y1): now also IC2.2 (I2)
- net at R23.2, SW2.1: now also A1.15 (D12); no longer A1.16 (D13)
- net at U3.15 (Y0): now also IC2.1 (I1)
- net at A1.13 (D10): now also R24.2, SW2.2
- net at U3.13 (Y2): now also IC2.3 (I3)
- net at R6.2: now also IC2.15 (O2)
- net at D8.1 (K), L1.1: now also IC1.2 (OUTPUT)
- net at R12.2: now also IC2.13 (O4)
- net at U3.12 (Y3): now also IC2.4 (I4)
- net at R1.2: now also IC2.16 (O1)
- net at R9.2: now also IC2.14 (O3)
- no-connect marks 20 -> 23
Other:
- moved on the sheet: BT1, BT2, C4, C5, C6, C7, D1, D2, D3, D4, D5, D8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
