File: micromouse-hardware.kicad_sch (KiCad schematic)
At the start: 46 parts, among them IC1 LM2575SX-5.0_NOPB, IC2 TBD62003AFG,EL, J1 BATT-CONN, Q4 TEFT4300, Q5 TEFT4300, Q6 TEFT4300, Q7 TEFT4300, Q8 TEFT4300, SW2 SW_DIP_x02, SW3 SLW-116641-5A-S-D, U1 DRV8833PWPR, U2 CD74HC4051M, U3 74HC238D

Commit message: PCB clean up
Changed lines of the file:
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@@
 	(wire
 		(pts
-			(xy 142.24 63.5) (xy 105.41 63.5)
+			(xy 142.24 59.055) (xy 105.41 59.055)
 		)
 		(stroke
@@
 	(wire
 		(pts
-			(xy 105.41 63.5) (xy 105.41 66.04)
+			(xy 105.41 59.055) (xy 105.41 66.04)
 		)
 		(stroke
@@
 	(wire
 		(pts
-			(xy 142.24 52.07) (xy 142.24 63.5)
-		)
-		(stroke
+			(xy 142.24 52.07) (xy 142.24 59.055)
+		)
+		(stroke

Commit message: kao gotov al da se poboljsat pcb
Parts:
- removed A1: Arduino_Nano_v3.x, Module:Arduino_Nano, symbol MCU_Module:Arduino_Nano_v3.x
- removed D5: SFH4545, LED_THT:LED_D5.0mm_Horizontal_O3.81mm_Z3.0mm, symbol Device:LED
- removed Q8: TEFT4300, LED_THT:LED_D3.0mm_Horizontal_O3.81mm_Z2.0mm, symbol Device:Q_Photo_NPN
- removed R15: 33R, Resistor_SMD:R_0805_2012Metric_Pad1.20x1.40mm_HandSolder, symbol Device:R
- removed R20: 1k8, Resistor_THT:R_Axial_DIN0207_L6.3mm_D2.5mm_P10.16mm_Horizontal, symbol Device:R
- removed R23, R24: 10K, Resistor_SMD:R_0805_2012Metric_Pad1.20x1.40mm_HandSolder, symbol Device:R
- removed SW2: SW_DIP_x02, Button_Switch_THT:SW_DIP_SPSTx02_Slide_9.78x7.26mm_W7.62mm_P2.54mm, symbol Switch:SW_DIP_x02
- added C11: 10uF, Capacitor_SMD:C_0805_2012Metric_Pad1.18x1.45mm_HandSolder, symbol Device:C
- added C13, C15: 2.2uF, Capacitor_SMD:C_0805_2012Metric_Pad1.18x1.45mm_HandSolder, symbol Device:C
- added C3, C5, C7, C8, C9: 100nF, Capacitor_SMD:C_0805_2012Metric_Pad1.18x1.45mm_HandSolder, symbol Device:C
- added J1: Conn_ARM_JTAG_SWD_10, Connector_PinHeader_1.27mm:PinHeader_2x05_P1.27mm_Vertical_SMD, symbol Connector:Conn_ARM_JTAG_SWD_10
- added R5, R6, R7: 10K, Resistor_SMD:R_0805_2012Metric_Pad1.20x1.40mm_HandSolder, symbol Device:R
- added SW1: SW_DIP_x02, Button_Switch_THT:SW_DIP_SPSTx02_Slide_9.78x7.26mm_W7.62mm_P2.54mm, symbol Switch:SW_DIP_x02
- added U2: STM32G431KBTx, Package_QFP:LQFP-32_7x7mm_P0.8mm, symbol MCU_ST_STM32G4:STM32G431KBTx
- added U3: LSM6DSO32TR, Package_LGA:LGA-14_3x2.5mm_P0.5mm_LayoutBorder3x4y, symbol Sensor_Motion:LSM6DS3
- added U6: TPS7A20xxxDBV, Package_TO_SOT_SMD:SOT-23-5, symbol Regulator_Linear:TPS7A20xxxDBV
- ME1, ME2: value ~ -> (none); footprint Connector_PinHeader_2.54mm:PinHeader_1x06_P2.54mm_Vertical -> Connector_PinHeader_2.54mm:PinHeader_1x06_P2.54mm_Vertical_SMD_Pin1Left
- renumbered C8 to C1, C9 to C12, C6 to C14, C5 to C16, C4 to C17, C7 to C18, C3 to C2, C2 to C4, C1 to C6, D8 to D5, IC2 to IC1, IC1 to IC2, J1 to J2, Q4 to Q1, Q5 to Q2, Q6 to Q3, Q7 to Q4, R18 to R10, R19 to R11, R6 to R2, R9 to R3, R12 to R4, R16 to R8, R17 to R9, SW3 to SW2, U3 to U1, U1 to U4, U2 to U5
Connections:
- net MUX_SEL_2 is gone; now on net GND: U1.3 (A2), U5.9 (S2)
- net +5V: now also C13.1, U6.1 (IN), U6.3 (EN); no longer C1.1, C12.1, D1.2 (A), D2.2 (A), D3.2 (A), D4.2 (A), IC1.9 (COMMON), ME1.5 (VCC), ME2.5 (VCC), Q1.1 (C), Q2.1 (C), Q3.1 (C), Q4.1 (C), U1.16 (VCC), U5.16 (VCC)
- net GND: now also C11.2, C13.2, C15.2, C3.2, C5.2, C7.2, C8.2, C9.2, J1.3 (GND), J1.5 (GND), J1.9 (GNDDetect), R5.1, R6.1, R7.1, U2.14 (VSSA), U2.16 (VSS), U2.32 (VSS), U3.6 (GND), U3.7 (GND), U6.2 (GND)
- net IRT_READ: now also U2.6 (PA1)
- net LED_DEMUX_ENABLE: now also U2.22 (PA12)
- net M1-C1: now also U2.11 (PA6)
- net M1-C2: now also U2.9 (PA4)
- net M1-IN1: now also U2.18 (PA8)
- net M1-IN2: now also U2.21 (PA11)
- net M2-C1: now also U2.29 (PB6)
- net M2-C2: now also U2.30 (PB7)
- net M2-IN1: now also U2.25 (PA15)
- net M2-IN2: now also U2.7 (PA2)
- net MUX_SEL_0: now also U2.19 (PA9)
- net MUX_SEL_1: now also U2.20 (PA10)
- net at IC1.5 (I5): no longer U1.11 (Y4)
- new net +3V3: C1.1, C11.1, C12.1, C15.1, C3.1, C5.1, C8.1, C9.1, D1.2 (A), D2.2 (A), D3.2 (A), D4.2 (A), IC1.9 (COMMON), J1.1 (VTref), ME1.5 (VCC), ME2.5 (VCC), Q1.1 (C), Q2.1 (C), Q3.1 (C), Q4.1 (C), SW1.3, SW1.4, U1.16 (VCC), U2.1 (VDD), U2.15 (VDDA), U2.17 (VDD), U3.5 (VDDIO), U3.8 (VDD), U5.16 (VCC), U6.5 (OUT)
- new net IMU_CS: U2.8 (PA3), U3.12 (CS)
- new net IMU_INT1: U2.5 (PA0), U3.4 (INT1)
- new net MCU_BOOT0: R6.2, U2.31 (PB8)
- new net MCU_NRESET: C7.1, J1.10 (~{RESET}), U2.4 (PG10)
- new net MCU_TCK: J1.4 (SWCLK/TCK), U2.24 (PA14)
- new net MCU_TDO: J1.6 (SWO/TDO), U2.26 (PB3)
- new net MCU_TMS: J1.2 (SWDIO/TMS), U2.23 (PA13)
- new net SPI1_CLK: U2.10 (PA5), U3.13 (SCL)
- new net SPI1_MISO: U2.27 (PB4), U3.1 (SDO/SA0)
- new net SPI1_MOSI: U2.28 (PB5), U3.14 (SDA)
- new net SW1: R5.2, SW1.2, U2.2 (PF0)
- new net SW2: R7.2, SW1.1, U2.3 (PF1)
- no-connect marks 23 -> 22
Other:
- note added: "3V3 LDO"
- note added: "IMU"
- note added: "MCU decouple"
- note added: "Switch"
- moved on the sheet: C1, C2, C4, C6, D1, D2, D3, D4, IC1, ME1, ME2, R1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
