File: micromouse-hardware.kicad_pcb (KiCad board)
At the start: 2 copper layers, 85 x 103.5 mm, 44 parts, among them IC1 LM2575SX-5.0_NOPB, IC2 TBD62003AFG,EL, J1 BATT-CONN, Q4 TEFT4300, Q5 TEFT4300, Q6 TEFT4300, Q7 TEFT4300, Q8 TEFT4300, SW2 SW_DIP_x02, SW3 SLW-116641-5A-S-D, U1 DRV8833PWPR, U2 CD74HC4051M, U3 74HC238D

Commit message: PCB clean up
Parts:
- moved C9 3.60 mm to (164.7, 73.7), turned to 90 degrees
- moved U2 0.81 mm to (157.5, 73.7)
- moved C5 0.75 mm to (175.8, 109.2)
- moved C2 0.28 mm to (149.0, 99.2)
- moved C3 0.15 mm to (153.4, 99.2)
- moved C1 0.09 mm to (151.3, 99.2)
Routing:
- net +5V: track 324.2 -> 356.7 mm, vias 5 -> 7
- net GND: track 16.2 -> 0.95 mm, vias 14 -> 321
- net +VBAT: track 92.7 -> 80.8 mm
- net /IRT_READ: track 43.8 -> 40.5 mm, vias 2 -> 1
- net Net-(Q7-E): track 50.2 -> 47.5 mm
- net Net-(IC2-O1): track 36.3 -> 37.5 mm
- net Net-(Q8-E): track 26.7 -> 25.9 mm
- net Net-(D1-K): track 6.88 -> 6.09 mm
- net /MUX_SEL_0: track 24.2 -> 23.5 mm
- net Net-(IC2-O5): track 38.9 -> 39.6 mm, vias 2 -> 0
- net Net-(A1-D10): track 41.7 -> 42.3 mm
- net /MUX_SEL_2: track 18.2 -> 17.6 mm

Commit message: kao gotov al da se poboljsat pcb
Parts:
- removed A1: Arduino_Nano_v3.x, Module:Arduino_Nano
- removed the D5 at (184.7, 86.8)
- removed Q8: TEFT4300, LED_THT:LED_D3.0mm_Horizontal_O3.81mm_Z2.0mm
- removed R15: 33R, Resistor_SMD:R_0805_2012Metric_Pad1.20x1.40mm_HandSolder
- removed R20: 1k8, Resistor_THT:R_Axial_DIN0207_L6.3mm_D2.5mm_P10.16mm_Horizontal
- removed R23, R24: 10K, Resistor_SMD:R_0805_2012Metric_Pad1.20x1.40mm_HandSolder
- removed the SW2 at (117.7, 99.7)
- added C11: 10uF, Capacitor_SMD:C_0805_2012Metric_Pad1.18x1.45mm_HandSolder, F.Cu at (134.0, 105.5)
- added C13: 2.2uF, Capacitor_SMD:C_0805_2012Metric_Pad1.18x1.45mm_HandSolder, F.Cu at (177.0, 91.5)
- added C15: 2.2uF, Capacitor_SMD:C_0805_2012Metric_Pad1.18x1.45mm_HandSolder, F.Cu at (174.0, 91.5)
- added C3: 100nF, Capacitor_SMD:C_0805_2012Metric_Pad1.18x1.45mm_HandSolder, B.Cu at (148.5, 131.5)
- added C5: 100nF, Capacitor_SMD:C_0805_2012Metric_Pad1.18x1.45mm_HandSolder, B.Cu at (151.5, 131.5)
- added C7: 100nF, Capacitor_SMD:C_0805_2012Metric_Pad1.18x1.45mm_HandSolder, F.Cu at (133.0, 108.5)
- added C8: 100nF, Capacitor_SMD:C_0805_2012Metric_Pad1.18x1.45mm_HandSolder, F.Cu at (145.5, 99.0)
- added C9: 100nF, Capacitor_SMD:C_0805_2012Metric_Pad1.18x1.45mm_HandSolder, F.Cu at (131.5, 105.5)
- added J1: Conn_ARM_JTAG_SWD_10, Connector_PinHeader_1.27mm:PinHeader_2x05_P1.27mm_Vertical_SMD, F.Cu at (112.0, 93.5)
- added R5: 10K, Resistor_SMD:R_0805_2012Metric_Pad1.20x1.40mm_HandSolder, F.Cu at (120.5, 98.5)
- added R6: 10K, Resistor_SMD:R_0805_2012Metric_Pad1.20x1.40mm_HandSolder, F.Cu at (128.0, 105.5)
- added R7: 10K, Resistor_SMD:R_0805_2012Metric_Pad1.20x1.40mm_HandSolder, F.Cu at (120.5, 101.5)
- added SW1: SW_DIP_x02, Button_Switch_THT:SW_DIP_SPSTx02_Slide_9.78x7.26mm_W7.62mm_P2.54mm, F.Cu at (117.0, 104.0)
- added U2: STM32G431KBTx, Package_QFP:LQFP-32_7x7mm_P0.8mm, F.Cu at (139.0, 100.0)
- added U3: LSM6DSO32TR, Package_LGA:LGA-14_3x2.5mm_P0.5mm_LayoutBorder3x4y, B.Cu at (150.1, 127.5)
- added U6: TPS7A20xxxDBV, Package_TO_SOT_SMD:SOT-23-5, F.Cu at (175.2, 86.5)
- D3: moved to B.Cu
- ME1, ME2: footprint Connector_PinHeader_2.54mm:PinHeader_1x06_P2.54mm_Vertical -> Connector_PinHeader_2.54mm:PinHeader_1x06_P2.54mm_Vertical_SMD_Pin1Left
- moved C14 62.1 mm to (154.1, 143.0)
- moved C12 33.7 mm to (131.0, 73.5)
- moved J2 30.6 mm to (166.5, 94.8), turned to -90 degrees
- moved R11 30.2 mm to (183.1, 70.2), turned to 180 degrees
- moved Q3 28.9 mm to (176.8, 58.4)
- moved D4 27.8 mm to (186.5, 85.6), turned to 125 degrees
- moved SW2 24.3 mm to (153.2, 94.8), turned to 90 degrees
- moved U5 22.9 mm to (136.5, 83.0), turned to 90 degrees
- moved R4 20.3 mm to (181.5, 82.2), turned to 90 degrees
- moved Q4 15.6 mm to (185.5, 79.0), turned to 125 degrees
- moved D3 15.2 mm to (168.2, 58.3), turned to 0 degrees
- moved R9 14.3 mm to (144.8, 48.0)
- moved U1 11.1 mm to (150.5, 83.0)
- moved R3 10.3 mm to (162.0, 58.0)
- moved C17 9.67 mm to (141.1, 143.0)
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- renumbered C8 to C1, C9 to C12, C6 to C14, C5 to C16, C4 to C17, C7 to C18, C3 to C2, C2 to C4, C1 to C6, D8 to D5, IC2 to IC1, IC1 to IC2, J1 to J2, Q4 to Q1, Q5 to Q2, Q6 to Q3, Q7 to Q4, R18 to R10, R19 to R11, R6 to R2, R9 to R3, R12 to R4, R16 to R8, R17 to R9, SW3 to SW2, U3 to U1, U1 to U4, U2 to U5
Connections:
- C1 pad 1: +5V -> +3V3
- C12 pad 1: +5V -> +3V3
- D1 pad 2: +5V -> +3V3
- D2 pad 2: +5V -> +3V3
- D3 pad 2: +5V -> +3V3
- D4 pad 2: +5V -> +3V3
- IC1 pad 12: Net-(IC2-O5) -> unconnected-(IC1-O5-Pad12)
- IC1 pad 5: Net-(IC2-I5) -> unconnected-(IC1-I5-Pad5)
- IC1 pad 9: +5V -> +3V3
- ME1 pad 5: +5V -> +3V3
- ME2 pad 5: +5V -> +3V3
- Q1 pad 1: +5V -> +3V3
- Q2 pad 1: +5V -> +3V3
- Q3 pad 1: +5V -> +3V3
- Q4 pad 1: +5V -> +3V3
- U1 pad 11: Net-(IC2-I5) -> unconnected-(U1-Y4-Pad11)
- U1 pad 16: +5V -> +3V3
- U1 pad 3: /MUX_SEL_2 -> GND
- U5 pad 1: Net-(Q8-E) -> unconnected-(U5-A4-Pad1)
- U5 pad 16: +5V -> +3V3
- U5 pad 9: /MUX_SEL_2 -> GND
Routing:
- net +3V3: track 0.00 -> 375.0 mm, vias 0 -> 12
- net +5V: track 356.7 -> 112.9 mm, vias 7 -> 3
- net /IMU_INT1: track 0.00 -> 57.6 mm, vias 0 -> 1
- net /M2-C1: track 37.3 -> 87.5 mm, vias 2 -> 0
- net Net-(A1-D10): track 42.3 -> 0.00 mm, vias 1 -> 0
- net /SPI1_MISO: track 0.00 -> 40.2 mm, vias 0 -> 3
- net Net-(IC2-O5): track 39.6 -> 0.00 mm
- net /SPI1_MOSI: track 0.00 -> 38.2 mm, vias 0 -> 3
- net /M2-C2: track 39.5 -> 77.4 mm, vias 2 -> 0
- net /MCU_NRESET: track 0.00 -> 35.1 mm, vias 0 -> 2
- net Net-(A1-D12): track 30.0 -> 0.00 mm
- net /SW2: track 0.00 -> 28.5 mm, vias 0 -> 1
- net /SW1: track 0.00 -> 28.1 mm, vias 0 -> 1
- net /SPI1_CLK: track 0.00 -> 27.9 mm, vias 0 -> 1
- net Net-(Q3-E): track 39.8 -> 66.8 mm, vias 1 -> 0
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Other:
- outline, holes or cut-outs redrawn
- board text removed: "By: Ian Petek & Erik Braun"
- board text removed: "JLCJLCJLC"
- board text removed: "XFER"
